Commit message: Add trajectory and goal publisher

File: src/hybrid_astar_planning/hybrid_astar_model/urdf/simple_car.urdf.xacro (robot description, xacro)
@@ -1,23 +1,42 @@
 <?xml version="1.0"?>
 <robot name="car" xmlns:xacro="http://www.ros.org/wiki/xacro">
-    <link name="world"/>
+    <link name="world" />
     <link name="base_link">
         <visual>
-            <origin xyz="0 0 0" rpy="${radians(90)} 0 0"/>
+            <origin xyz="0 0 0" rpy="${radians(90)} 0 0" />
             <geometry>
-                <mesh filename="file:///$(find hybrid_astar_model)/meshes/car.dae"/>
+                <mesh filename="file:///$(find hybrid_astar_model)/meshes/car.dae" />
             </geometry>
         </visual>
         <collision>
-            <origin xyz="0 0 0" rpy="${radians(90)} 0 0"/>
+            <origin xyz="0 0 0" rpy="${radians(90)} 0 0" />
             <geometry>
-                <mesh filename="file:///$(find hybrid_astar_model)/meshes/car.dae"/>
+                <mesh filename="file:///$(find hybrid_astar_model)/meshes/car.dae" />
             </geometry>
         </collision>
     </link>
-    <joint name="base_joint" type="fixed">
-        <parent link="world"/>
-        <child link="base_link"/>
-        <origin xyz="0 0 0" rpy="0 0 0"/>
+    <link name="base_link_2">
+        <visual>
+            <origin xyz="0 0 0" rpy="${radians(90)} 0 0" />
+            <geometry>
+                <mesh filename="file:///$(find hybrid_astar_model)/meshes/car.dae" />
+            </geometry>
+        </visual>
+        <collision>
+            <origin xyz="0 0 0" rpy="${radians(90)} 0 0" />
+            <geometry>
+                <mesh filename="file:///$(find hybrid_astar_model)/meshes/car.dae" />
+            </geometry>
+        </collision>
+    </link>
+    <joint name="base_joint_1" type="fixed">
+        <parent link="world" />
+        <child link="base_link" />
+        <origin xyz="0 0 0" rpy="0 0 0" />
+    </joint>
+    <joint name="base_joint_2" type="fixed">
+        <parent link="world" />
+        <child link="base_link_2" />
+        <origin xyz="0 0 0" rpy="0 0 0" />
     </joint>
 </robot>
